File: pico_test_w5100s_evb.brd (EAGLE design)
At the start: 100 x 100 mm, 22 parts, among them U1 MAX485ESA+T, U2 MAX485ESA+T

Commit message: gerber
Parts:
- moved R4 8.62 mm to (25.3, 28.3), turned to 180 degrees
- moved R6 7.73 mm to (11.8, 31.6)
- moved U$9 7.73 mm to (14.5, 31.6)
- moved R3 7.62 mm to (23.3, 31.2)
- moved U1 7.62 mm to (24.1, 20.1)
- moved U2 7.62 mm to (12.7, 20.0)
- moved U$7 7.62 mm to (26.0, 31.2)
- moved R7 7.03 mm to (15.6, 28.3), turned to 0 degrees
- moved U$1 5.08 mm to (37.4, 73.7)
Connections:
- net GND: now also U$1.P$13, U$1.P$18, U$1.P$23, U$1.P$28, U$1.P$3, U$1.P$33, U$1.P$38, U$1.P$8
Routing:
- net N$8: track 51.7 -> 0.00 mm
- net 485_1_DI: track 56.3 -> 80.0 mm
- net +5V: track 117.7 -> 140.5 mm
- net 485_1_RO: track 46.9 -> 69.2 mm
- net 485_2_RO: track 28.6 -> 44.8 mm
- net GND: track 0.00 -> 14.5 mm, vias 0 -> 24
- net 485_2_DI: track 38.8 -> 53.1 mm
- net 485_1_DE: track 52.4 -> 65.1 mm
- net 485_2_DE: track 32.8 -> 44.0 mm
- net N$6: track 13.3 -> 19.5 mm
- net N$10: track 13.3 -> 19.4 mm
- net N$11: track 13.2 -> 19.3 mm
- net N$7: track 13.3 -> 19.3 mm
- net N$4: track 43.3 -> 45.5 mm
- net +3V3: track 71.6 -> 73.5 mm
Other:
- outline, holes or cut-outs redrawn
