File: pico_test_w5100s_evb.sch (EAGLE design)
At the start: 22 parts, among them U1 MAX485ESA+T, U2 MAX485ESA+T

Commit message: gerber
Connections:
- net GND: now also U$1.GND
Changed lines of the file:
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@@
 <part name="+3V3" library="picoRS485Gateway" deviceset="+3V3" device=""/>
 <part name="P+4" library="picoRS485Gateway" deviceset="+5V" device=""/>
+<part name="GND4" library="picoRS485Gateway" deviceset="GND" device=""/>
 </parts>
 <sheets>
@@
 <instance part="P+4" gate="1" x="177.8" y="142.24" smashed="yes">
 <attribute name="VALUE" x="175.26" y="139.7" size="1.778" layer="96" rot="R90"/>
+</instance>
+<instance part="GND4" gate="1" x="180.34" y="76.2" smashed="yes">
+<attribute name="VALUE" x="177.8" y="73.66" size="1.778" layer="96"/>
 </instance>
 </instances>
@@
 <wire x1="281.94" y1="203.2" x2="294.64" y2="203.2" width="0.1524" layer="91"/>
 </segment>
-</net>
+<segment>
+<pinref part="GND4" gate="1" pin="GND"/>
+<pinref part="U$1" gate="G$1" pin="GND"/>
+<wire x1="180.34" y1="78.74" x2="180.34" y2="81.28" width="0.1524" layer="91"/>
+</segment>
+</net>
